File: kicad/TeaSteaper.kicad_pcb (KiCad board)
At the start: 2 copper layers, 100 x 60 mm, 16 parts, among them J1 Serial, J2 JTAG, J3 Barrel_Jack_Switch, J4 Display, J5 Conn_01x05, SW2 Rotary_Encoder_Switch, U1 ESP32-WROOM-32D, U2 ULN2803A, U3 AH3572-SA-7, U5 AZ1117-3.3

Commit message: board v1.0 ordered
Parts:
- J3: value Barrel_Jack_Switch -> Power +5v
- J4: footprint TeaMaker:JST_PH_S8B-PH-K_1x08_P2.00mm_Horizontal -> TeaMaker:JST_PH_B8B-PH-K_1x08_P2.00mm_Vertical; moved to B.Cu
- J5: value Conn_01x05 -> Stepper
- moved C5 52.2 mm to (159.0, 152.6), turned to 270 degrees
- moved C4 49.4 mm to (155.2, 152.7), turned to 270 degrees
- moved J4 39.9 mm to (124.2, 149.5), turned to 180 degrees
- moved U1 33.3 mm to (142.8, 145.0), turned to 180 degrees
- moved U2 30.1 mm to (173.0, 133.8)
- moved C3 28.7 mm to (97.7, 130.8), turned to 270 degrees
- moved C1 28.1 mm to (97.7, 116.3), turned to 90 degrees
- moved R1 26.2 mm to (97.7, 122.5), turned to 90 degrees
- moved U5 26.1 mm to (103.0, 132.8), turned to 90 degrees
- moved J2 25.5 mm to (120.7, 112.8), turned to 0 degrees
- moved SW2 18.0 mm to (135.2, 118.8)
- moved C2 15.5 mm to (108.3, 134.9), turned to 90 degrees
- moved J1 8.07 mm to (105.5, 113.3), turned to 0 degrees
- moved U3 3.00 mm to (179.0, 116.3)
- moved J5 2.42 mm to (177.7, 148.9), turned to 0 degrees
Connections:
- J4 pad 1: +3V3 -> /BL
- J4 pad 2: GND -> /RST
- J4 pad 3: /MOSI -> /DC
- J4 pad 4: /SCLK -> /CS
- J4 pad 5: /CS -> /SCLK
- J4 pad 6: /DC -> /MOSI
- J4 pad 7: /RST -> GND
- J4 pad 8: /BL -> +3V3
Routing:
- net /EN: track 40.0 -> 98.9 mm
- net /RST: track 56.8 -> 12.6 mm
- net /TXD: track 11.3 -> 48.4 mm, vias 0 -> 2
- net /ROTSW: track 56.5 -> 22.7 mm
- net /RXD: track 11.8 -> 44.7 mm, vias 0 -> 2
- net +3V3: track 113.2 -> 144.4 mm, vias 1 -> 2
- net /DC: track 44.9 -> 15.1 mm
- net /TMS: track 16.6 -> 44.5 mm, vias 0 -> 2
- net /MOSI: track 48.4 -> 21.1 mm
- net /BL: track 42.1 -> 17.9 mm, vias 2 -> 1
- net /TCK: track 11.8 -> 35.5 mm, vias 0 -> 2
- net /SCLK: track 46.1 -> 22.4 mm
- net /CS: track 40.2 -> 19.2 mm
- net +5V: track 91.1 -> 107.3 mm
- net /TDO: track 12.8 -> 28.8 mm, vias 0 -> 2
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Other:
- outline, holes or cut-outs redrawn
- net class Default: clearance 0.2 -> 0.15; trace_width 0.25 -> 0.16
- rule trace_clearance: 0.2 -> 0.15
- rule trace_min: 0.2 -> 0.15
- board text added: "Tea Steaper 1.0 Designed By Christopher B. Liebman"

Commit message: board v1.1
Parts:
- moved C5 91.8 mm to (191.0, 66.6), turned to 0 degrees
- moved C4 89.8 mm to (191.1, 70.4), turned to 0 degrees
- moved U2 77.4 mm to (153.3, 59.0), turned to 180 degrees
- moved J4 75.3 mm to (184.1, 103.9), turned to 270 degrees
- moved U1 74.2 mm to (184.2, 83.4), turned to 270 degrees
- moved J5 73.8 mm to (138.6, 86.3), turned to 90 degrees
- moved J1 67.3 mm to (171.2, 127.9), turned to 90 degrees
- moved C1 63.0 mm to (160.2, 123.9)
- moved R1 63.0 mm to (160.2, 130.1)
- moved U3 61.4 mm to (180.5, 54.9)
- moved C3 57.7 mm to (146.7, 100.4), turned to 180 degrees
- moved U5 49.8 mm to (144.7, 105.6), turned to 0 degrees
- moved J3 48.4 mm to (144.2, 122.9)
- moved J2 43.4 mm to (150.4, 81.2)
- moved C2 41.8 mm to (142.5, 111.0), turned to 0 degrees
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Connections:
- J5 pad 1: +5V -> /P_M1A
- J5 pad 2: /P_M1D -> /P_M1B
- J5 pad 4: /P_M1B -> /P_M1D
- J5 pad 5: /P_M1A -> +5V
Routing:
- net +5V: track 107.3 -> 79.7 mm
- net +3V3: track 144.4 -> 169.2 mm, vias 2 -> 1
- net /ULIM: track 69.4 -> 45.9 mm
- net /IO0: track 34.5 -> 52.0 mm
- net /M1D: track 21.2 -> 38.5 mm
- net /TMS: track 44.5 -> 28.7 mm, vias 2 -> 0
- net /P_M1D: track 14.9 -> 28.7 mm
- net /TCK: track 35.5 -> 24.0 mm, vias 2 -> 0
- net /P_M1C: track 18.5 -> 29.1 mm
- net GND: track 8.04 -> 0.00 mm, vias 24 -> 11
- net /P_M1B: track 21.4 -> 29.3 mm
- net /ROTA: track 28.0 -> 20.9 mm, vias 0 -> 2
- net /TDO: track 28.8 -> 22.7 mm, vias 2 -> 0
- net /ROTSW: track 22.7 -> 28.6 mm, vias 0 -> 1
- net /RST: track 12.6 -> 16.4 mm
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Other:
- board size 100 x 60 mm -> 60 x 100 mm
- board text added: "Tea Steeper 1.1 Designed By Christopher B. Liebman"
- board text removed: "Tea Steaper 1.0 Designed By Christopher B. Liebman"
