File: kicad/TeaSteaper.sch (KiCad schematic (older format))
At the start: 16 parts, among them J1 Serial, J2 JTAG, J3 Barrel_Jack_Switch, J4 Display, J5 Conn_01x05, SW2 Rotary_Encoder_Switch, U1 ESP32-WROOM-32D, U2 ULN2803A, U3 AH3572-SA-7, U5 AZ1117-3.3

Commit message: board v1.0 ordered
Parts:
- J3: value Barrel_Jack_Switch -> Power +5v
- J4: footprint TeaMaker:JST_PH_S8B-PH-K_1x08_P2.00mm_Horizontal -> TeaMaker:JST_PH_B8B-PH-K_1x08_P2.00mm_Vertical
- J5: value Conn_01x05 -> Stepper
Connections:
- net +3V3: now also J4.8 (Pin_8); no longer J4.1 (Pin_1)
- net BL: now also J4.1 (Pin_1); no longer J4.8 (Pin_8)
- net CS: now also J4.4 (Pin_4); no longer J4.5 (Pin_5)
- net DC: now also J4.3 (Pin_3); no longer J4.6 (Pin_6)
- net GND: now also J4.7 (Pin_7); no longer J4.2 (Pin_2)
- net MOSI: now also J4.6 (Pin_6); no longer J4.3 (Pin_3)
- net RST: now also J4.2 (Pin_2); no longer J4.7 (Pin_7)
- net SCLK: now also J4.5 (Pin_5); no longer J4.4 (Pin_4)
Changed lines of the file:
@@
 P 1700 6100
 F 0 "J3" H 1757 6417 50  0000 C CNN
-F 1 "Barrel_Jack_Switch" H 1757 6326 50  0000 C CNN
+F 1 "Power +5v" H 1757 6326 50  0000 C CNN
 F 2 "TeaMaker:BarrelJack_CUI_PJ-202A_Horizontal" H 1750 6060 50  0001 C CNN
 F 3 "~" H 1750 6060 50  0001 C CNN
@@
 L TeaSteaper:Conn_01x08 J4
 U 1 1 6181980D
-P 9450 1300
-F 0 "J4" H 9530 1292 50  0000 L CNN
-F 1 "Display" H 9530 1201 50  0000 L CNN
-F 2 "TeaMaker:JST_PH_S8B-PH-K_1x08_P2.00mm_Horizontal" H 9450 1300 50  0001 C CNN
-F 3 "~" H 9450 1300 50  0001 C CNN
-	1    9450 1300
-	1    0    0    -1
+P 9450 1400
+F 0 "J4" H 9530 1392 50  0000 L CNN
+F 1 "Display" H 9530 1301 50  0000 L CNN
+F 2 "TeaMaker:JST_PH_B8B-PH-K_1x08_P2.00mm_Vertical" H 9450 1400 50  0001 C CNN
+F 3 "~" H 9450 1400 50  0001 C CNN
+	1    9450 1400
+	1    0    0    1
 $EndComp
 Wire Wire Line
@@
 P 9250 5250
 F 0 "J5" H 9330 5292 50  0000 L CNN
-F 1 "Conn_01x05" H 9330 5201 50  0000 L CNN
+F 1 "Stepper" H 9330 5201 50  0000 L CNN
 F 2 "TeaMaker:JST_XH_B5B-XH-A_1x05_P2.50mm_Vertical" H 9250 5250 50  0001 C CNN
 F 3 "~" H 9250 5250 50  0001 C CNN

Commit message: board v1.1
Connections:
- net +5V: now also J5.5 (Pin_5); no longer J5.1 (Pin_1)
- net P_M1A: now also J5.1 (Pin_1); no longer J5.5 (Pin_5)
- net P_M1B: now also J5.2 (Pin_2); no longer J5.4 (Pin_4)
- net P_M1D: now also J5.4 (Pin_4); no longer J5.2 (Pin_2)
Changed lines of the file:
@@
 encoding utf-8
 Sheet 1 1
-Title "TeaSteaper"
-Date "2021-10-21"
-Rev "1.0"
+Title "TeaSteeper"
+Date "2021-11-03"
+Rev "1.1"
 Comp "Christopher B. Liebman"
 Comment1 ""
@@
 F 3 "~" H 9250 5250 50  0001 C CNN
 	1    9250 5250
-	1    0    0    -1
-$EndComp
-Wire Wire Line
+	1    0    0    1
+$EndComp
+Wire Wire Line
